File: 26th_PCB_PitchSender.kicad_sch (KiCad schematic)
At the start: 14 parts, among them J1 vol, J2 Conn_01x04_Pin, J3 microSD, J4 Conn_01x04_Socket, J5 BNO055, J6 BMP390

Commit message: ESP32とスピーカー場所交代
Parts:
- J1: value vol -> Amp
- RV1: value R_Potentiometer -> Vol
Connections:
- net GND: now also U1.J2_14 (GND_J2_14)
- no-connect marks 31 -> 30
Changed lines of the file:
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@@
-	)
-	(no_connect
-		(at 144.78 127)
 	)
 	(no_connect
@@
 		(pts
 			(xy 82.55 144.78) (xy 82.55 161.29)
+		)
+		(stroke
+			(width 0)
+			(type default)
+		)
+	)
+	(wire
+		(pts
+			(xy 138.43 127) (xy 144.78 127)
 		)
 		(stroke
@@
 	)
 	(symbol
+		(lib_id "power:GND")
+		(at 138.43 127 270)
+		(unit 1)
+		(exclude_from_sim no)
+		(in_bom yes)
+		(on_board yes)
+		(dnp no)
+		(property "Reference" "#PWR018"
+			(at 132.08 127 0)
+			(effects
+				(font
+					(size 1.27 1.27)
+				)
+				(hide yes)
+			)
+		)
+		(property "Value" "GND"
+			(at 133.35 127 0)
+			(effects
+				(font
+					(size 1.27 1.27)
+				)
+			)
+		)
+		(property "Footprint" ""
+			(at 138.43 127 0)
+			(effects
+				(font
+					(size 1.27 1.27)
+				)
+				(hide yes)
+			)
+		)
+		(property "Datasheet" ""
+			(at 138.43 127 0)
+			(effects
+				(font
+					(size 1.27 1.27)
+				)
+				(hide yes)
+			)
+		)
+		(property "Description" "Power symbol creates a global label with name \"GND\" , ground"
+			(at 138.43 127 0)
+			(effects
+				(font
+					(size 1.27 1.27)
+				)
+				(hide yes)
+			)
+		)
+		(pin "1"
+		)
+		(instances
+			(project "26th_PCB_PitchSender"
+				(path "/5013cac2-53c1-4b5b-9014-63fb93daa52f"
+					(reference "#PWR018")
+					(unit 1)
+				)
+			)
+		)
+	)
+	(symbol
 		(lib_id "power:+3V3")
 		(at 222.25 78.74 0)
@@
 			)
 		)
-		(property "Value" "R_Potentiometer"
+		(property "Value" "Vol"
 			(at 93.98 167.64 90)
 			(effects
@@
 			)
 		)
-		(property "Value" "vol"
+		(property "Value" "Amp"
 			(at 73.025 139.7 0)
 			(effects
